File: hardware/f-ramune.sch (KiCad schematic (older format))
At the start: 3 parts, among them U1 Teensy3.2, U2 74HC595, U3 FM1808B-SG

Commit message: Rename project to f-ramune!
Enough work has gone into this that it shouldn't have a generic name.
Parts:
- U1: footprint (none) -> Housings_DIP:DIP-28_W7.62mm_Socket_LongPads
Changed lines of the file:
@@
 EESchema Schematic File Version 2
-LIBS:framtest
+LIBS:f-ramune
+LIBS:teensy
 LIBS:power
 LIBS:device
@@
 LIBS:contrib
 LIBS:valves
-LIBS:teensy
-LIBS:framtest-cache
 EELAYER 25 0
 EELAYER END
@@
 F 0 "U1" H 2950 4150 60  0000 C CNN
 F 1 "Teensy3.2" H 2950 1150 60  0000 C CNN
-F 2 "" H 2950 1850 60  0000 C CNN
+F 2 "Housings_DIP:DIP-28_W7.62mm_Socket_LongPads" H 2950 1050 60  0001 C CNN
 F 3 "" H 2950 1850 60  0000 C CNN
 	1    2950 2650
