File: hardware/pcb_avr/f-ramune_avr.kicad_pcb (KiCad board)
At the start: 2 copper layers, 63.5 x 45.5 mm, 27 parts, among them J1 ISP Header, J2 USB Type-B Port, Q1 IRL520N, SW1 SW_Push, U1 74HC595, U2 74HC595, U3 FRAM Socket (DIP-28), U4 ATmega328P-AU, U5 MCP2221A, Y1 16Mhz

Commit message: Fix incorrect copyright date on AVR silkscreen.
Other:
- board text added: "F-Ramune 1.0 ©2019 obskyr Designed in Sweden https://github.com/obskyr/f-ramune/ Insert chip into socket. Press button to test. GREEN: FRAM is genuine. GREEN+RED: FRAM is faulty. RED: FRAM is counterfeit."
- board text removed: "F-Ramune 1.0 ©2018 obskyr Designed in Sweden https://github.com/obskyr/f-ramune/ Insert chip into socket. Press button to test. GREEN: FRAM is genuine. GREEN+RED: FRAM is faulty. RED: FRAM is counterfeit."
Changed lines of the file:
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@@
     (solder_mask_min_width 0.25)
     (aux_axis_origin 0 0)
-    (visible_elements FFFFFF7F)
+    (visible_elements 7FFFFFFF)
     (pcbplotparams
       (layerselection 0x010fc_ffffffff)
@@
       (outputformat 1)
       (mirror false)
-      (drillshape 1)
+      (drillshape 0)
       (scaleselection 1)
-      (outputdirectory ""))
+      (outputdirectory "gerber/"))
   )
   (net 0 "")
@@
     (effects (font (size 1 1) (thickness 0.15)) (justify left mirror))
   )
-  (gr_text "F-Ramune 1.0 ©2018 obskyr\nDesigned in Sweden\nhttps://github.com/obskyr/f-ramune/\n\nInsert chip into socket. Press button to test.\nGREEN: FRAM is genuine.\nGREEN+RED: FRAM is faulty.\nRED: FRAM is counterfeit." (at 160.528 101.854) (layer B.SilkS)
+  (gr_text "F-Ramune 1.0 ©2019 obskyr\nDesigned in Sweden\nhttps://github.com/obskyr/f-ramune/\n\nInsert chip into socket. Press button to test.\nGREEN: FRAM is genuine.\nGREEN+RED: FRAM is faulty.\nRED: FRAM is counterfeit." (at 160.528 101.854) (layer B.SilkS)
     (effects (font (size 1 1) (thickness 0.15)) (justify left mirror))
   )
@@
   (gr_line (start 166.878 128.27) (end 105.156 128.27) (layer Edge.Cuts) (width 0.05))
   (gr_line (start 166.878 84.836) (end 166.878 128.27) (layer Edge.Cuts) (width 0.05))
-  (via (at 132.715 108.966) (size 0.8) (drill 0.4) (layers F.Cu B.Cu) (net 5))
-  (via (at 134.239 103.124) (size 0.8) (drill 0.4) (layers F.Cu B.Cu) (net 5))
-  (via (at 143.637 95.758) (size 0.8) (drill 0.4) (layers F.Cu B.Cu) (net 46))
-  (via (at 140.335 86.741) (size 0.8) (drill 0.4) (layers F.Cu B.Cu) (net 45))
-  (via (at 147.701 91.186) (size 0.8) (drill 0.4) (layers F.Cu B.Cu) (net 45))
-  (via (at 161.417 107.442) (size 0.8) (drill 0.4) (layers F.Cu B.Cu) (net 3))
-  (via (at 151.511 91.694) (size 0.8) (drill 0.4) (layers F.Cu B.Cu) (net 10))
-  (via (at 154.305 116.713) (size 0.8) (drill 0.4) (layers F.Cu B.Cu) (net 10))
-  (via (at 150.495 116.205) (size 0.8) (drill 0.4) (layers F.Cu B.Cu) (net 12))
-  (via (at 133.858 123.19) (size 0.8) (drill 0.4) (layers F.Cu B.Cu) (net 22))
-  (via (at 151.892 116.713) (size 0.8) (drill 0.4) (layers F.Cu B.Cu) (net 2))
-  (via (at 140.589 118.745) (size 0.8) (drill 0.4) (layers F.Cu B.Cu) (net 2))
-  (via (at 127.889 124.587) (size 0.8) (drill 0.4) (layers F.Cu B.Cu) (net 27))
   (segment (start 163.333 86.289) (end 163.333 88.763873) (width 0.25) (layer F.Cu) (net 1))
   (segment (start 161.836081 91.048) (end 163.333 91.048) (width 0.25) (layer F.Cu) (net 1))
@@
   (segment (start 157.390995 92.234001) (end 159.733001 92.234001) (width 0.25) (layer F.Cu) (net 1))
   (segment (start 150.681 97.898) (end 151.726996 97.898) (width 0.25) (layer F.Cu) (net 1))
+  (via (at 151.892 116.713) (size 0.8) (drill 0.4) (layers F.Cu B.Cu) (net 2))
+  (via (at 140.589 118.745) (size 0.8) (drill 0.4) (layers F.Cu B.Cu) (net 2))
   (segment (start 118.471 88.9) (end 122.301 88.9) (width 0.25) (layer B.Cu) (net 2))
   (segment (start 117.221 88.9) (end 118.471 88.9) (width 0.25) (layer B.Cu) (net 2))
@@
   (segment (start 158.623 89.959) (end 158.623 86.36) (width 0.25) (layer B.Cu) (net 2))
   (segment (start 158.623 86.36) (end 156.083 83.82) (width 0.25) (layer B.Cu) (net 2))
+  (via (at 161.417 107.442) (size 0.8) (drill 0.4) (layers F.Cu B.Cu) (net 3))
   (segment (start 162.447 108.472) (end 161.417 107.442) (width 0.25) (layer F.Cu) (net 3))
   (segment (start 162.447 108.966) (end 162.447 108.472) (width 0.25) (layer F.Cu) (net 3))
@@
   (segment (start 134.239 101.59999) (end 137.935578 101.59999) (width 0.25) (layer B.Cu) (net 4))
   (via (at 137.95899 101.623402) (size 0.8) (drill 0.4) (layers F.Cu B.Cu) (net 4))
+  (via (at 132.715 108.966) (size 0.8) (drill 0.4) (layers F.Cu B.Cu) (net 5))
+  (via (at 134.239 103.124) (size 0.8) (drill 0.4) (layers F.Cu B.Cu) (net 5))
   (segment (start 135.777 103.124) (end 134.239 103.124) (width 0.25) (layer F.Cu) (net 5))
   (segment (start 132.715 109.531685) (end 132.715 108.966) (width 0.25) (layer F.Cu) (net 5))
@@
   (segment (start 141.069 111.492) (end 141.478 111.492) (width 0.25) (layer F.Cu) (net 9))
   (segment (start 139.319 109.742) (end 141.069 111.492) (width 0.25) (layer F.Cu) (net 9))
+  (via (at 151.511 91.694) (size 0.8) (drill 0.4) (layers F.Cu B.Cu) (net 10))
+  (via (at 154.305 116.713) (size 0.8) (drill 0.4) (layers F.Cu B.Cu) (net 10))
   (segment (start 145.777 90.556) (end 145.777 93.794) (width 0.25) (layer F.Cu) (net 10))
   (segment (start 146.29 90.043) (end 145.777 90.556) (width 0.25) (layer F.Cu) (net 10))
@@
   (segment (start 148.177 102.802) (end 148.177 106.839006) (width 0.25) (layer F.Cu) (net 11))
   (segment (start 148.209 112.141) (end 148.082 112.014) (width 0.25) (layer B.Cu) (net 11))
+  (via (at 150.495 116.205) (size 0.8) (drill 0.4) (layers F.Cu B.Cu) (net 12))
   (segment (start 149.352 117.348) (end 150.495 116.205) (width 0.25) (layer F.Cu) (net 12))
   (segment (start 149.352 119.982) (end 149.352 117.348) (width 0.25) (layer F.Cu) (net 12))
@@
   (segment (start 136.906 125.89) (end 136.906 125.19) (width 0.25) (layer F.Cu) (net 21))
   (segment (start 104.775 125.986822) (end 104.775 95.986) (width 0.25) (layer F.Cu) (net 21))
+  (via (at 133.858 123.19) (size 0.8) (drill 0.4) (layers F.Cu B.Cu) (net 22))
   (segment (start 108.351 96.52) (end 107.061 96.52) (width 0.25) (layer B.Cu) (net 22))
   (segment (start 109.601 96.52) (end 108.351 96.52) (width 0.25) (layer B.Cu) (net 22))
@@
   (segment (start 130.556 125.19) (end 129.667 124.301) (width 0.25) (layer F.Cu) (net 26))
   (segment (start 129.667 124.517685) (end 129.667 123.952) (width 0.25) (layer B.Cu) (net 26))
+  (via (at 127.889 124.587) (size 0.8) (drill 0.4) (layers F.Cu B.Cu) (net 27))
   (segment (start 108.311 109.22) (end 109.601 109.22) (width 0.25) (layer B.Cu) (net 27))
   (segment (start 107.061 109.22) (end 108.311 109.22) (width 0.25) (layer B.Cu) (net 27))
@@
   (segment (start 138.049 106.934) (end 130.876322 106.934) (width 0.25) (layer F.Cu) (net 44))
   (segment (start 130.876322 106.934) (end 130.032334 107.777988) (width 0.25) (layer F.Cu) (net 44))
+  (via (at 140.335 86.741) (size 0.8) (drill 0.4) (layers F.Cu B.Cu) (net 45))
+  (via (at 147.701 91.186) (size 0.8) (drill 0.4) (layers F.Cu B.Cu) (net 45))
   (segment (start 117.221 104.14) (end 122.301 104.14) (width 0.25) (layer B.Cu) (net 45))
   (segment (start 146.577 92.31) (end 147.701 91.186) (width 0.25) (layer F.Cu) (net 45))
@@
   (segment (start 127 103.123998) (end 126.383997 103.740001) (width 0.25) (layer F.Cu) (net 45))
   (via (at 125.983998 104.14) (size 0.8) (drill 0.4) (layers F.Cu B.Cu) (net 45))
+  (via (at 143.637 95.758) (size 0.8) (drill 0.4) (layers F.Cu B.Cu) (net 46))
   (segment (start 117.221 91.44) (end 122.301 91.44) (width 0.25) (layer B.Cu) (net 46))
   (segment (start 122.581 91.44) (end 126.518 95.377) (width 0.25) (layer F.Cu) (net 46))
